File: kicad/buttons.sch (KiCad schematic (older format))
At the start: 6 parts, among them U1 74HC14

Commit message: Final routing
Removed some intermediary routing steps, too
Other:
- note added: "Return ground line from buttons"
- note added: "To board ground"
- note added: "To switches on front panel"
- note added: "Unused IC element"
- moved on the sheet: R14, R15, R16, R17, R18, U1A, U1B, U1C, U1D, U1E, U1F
