File: kicad/IO.sch (KiCad schematic (older format))
At the start: 6 parts, among them P3 CONN_02X12, P4 CONN_2, P5 CONN_3, P6 CONN_2

Commit message: Final routing
Removed some intermediary routing steps, too
Parts:
- removed R19: R, ~, symbol R
Connections:
- net labels removed: AudioIn, PA4
- wire segments 12 -> 7
Changed lines of the file:
@@
 Sheet 5 5
 Title ""
-Date "18 jun 2015"
+Date "19 jun 2015"
 Rev ""
 Comp ""
@@
 S5
 NoConn ~ 6150 2750
-Text GLabel 8750 1150 0    60   Input ~ 0
-AudioIn
-Wire Wire Line
-	8750 1150 9250 1150
-Wire Wire Line
-	9250 850  9250 1550
-Wire Wire Line
-	9250 850  9650 850
-Wire Wire Line
-	9800 1550 10200 1550
-Connection ~ 9250 1150
-Text GLabel 9650 850  2    60   Output ~ 0
-PA4
-Text GLabel 10200 1550 2    60   Output ~ 0
-AudiojackOut
 $Comp
 L CONN_2 P6
@@
 AudioJackGrnd
 $Comp
-L R R19
-U 1 1 557F4CDA
-P 9550 1550
-F 0 "R19" V 9630 1550 40  0000 C CNN
-F 1 "R" V 9557 1551 40  0000 C CNN
-F 2 "~" V 9480 1550 30  0000 C CNN
-F 3 "~" H 9550 1550 30  0000 C CNN
-	1    9550 1550
-	0    -1   -1   0
-$EndComp
-Wire Wire Line
-	9250 1550 9300 1550
-$Comp
 L STM32_F4_DISCOVERY STM1

Commit message: *Fix* Missing IO pins
Added PA4 to the schematic IO page and fixed PD8, PD10
Connections:
- net labels added: PA4
- wire segments 7 -> 9
- no-connect marks 85 -> 84
Changed lines of the file:
@@
 Sheet 5 5
 Title ""
-Date "19 jun 2015"
+Date "30 jun 2015"
 Rev ""
 Comp ""
@@
 Text GLabel 4100 3900 2    30   Input ~ 0
 PE13
-Text GLabel 2000 3000 0    30   Output ~ 0
+Text GLabel 4100 2300 2    30   Output ~ 0
 PD8
 Text GLabel 3900 2350 2    30   Output ~ 0
 PD9
-Text GLabel 2000 3100 0    30   Output ~ 0
+Text GLabel 4100 2400 2    30   Output ~ 0
 PD10
 Text GLabel 3900 2450 2    30   Output ~ 0
@@
 NoConn ~ 2000 3800
 NoConn ~ 2000 3750
-NoConn ~ 2000 3700
 NoConn ~ 2000 3650
 NoConn ~ 2000 3600
@@
 NoConn ~ 3900 2100
 NoConn ~ 3900 2150
-NoConn ~ 3900 2300
-NoConn ~ 3900 2400
 NoConn ~ 3900 2500
 NoConn ~ 3900 2550
@@
 Text GLabel 3200 1500 1    30   Output ~ 0
 3V_205
+NoConn ~ 2000 3000
+NoConn ~ 2000 3100
+Wire Wire Line
+	3900 2300 4100 2300
+Wire Wire Line
+	3900 2400 4100 2400
+Text GLabel 2000 3700 0    30   Output ~ 0
+PA4
 $EndSCHEMATC
